File: KBLE60.kicad_pcb (KiCad board)
At the start: 2 copper layers, 91 parts, among them J1 USB_C_Receptacle, J2 Ext_pin, J3 Debug, J4 Battery, Q1 Q_Dual_NMOS_G1S2G2D2S1D1, SW1 SW_Push, SW10 SW_DPDT_x2, SW11 SW_Push, SW12 SW_Push, SW13 SW_Push, SW14 SW_Push, SW15 SW_Push, SW16 SW_Push, SW17 SW_Push, SW18 SW_Push, SW19 SW_Push, SW2 SW_Push, SW20 SW_Push, SW21 SW_Push, SW22 SW_Push, SW23 SW_Push, SW24 SW_Push, SW25 SW_Push, SW26 SW_Push, SW27 SW_Push, SW28 SW_Push, SW29 SW_Push, SW3 SW_Push, SW30 SW_Push, SW31 SW_Push, SW32 SW_Push, SW33 SW_Push, SW34 SW_Push, SW35 SW_Push, SW36 SW_Push, SW37 SW_Push, SW38 SW_Push, SW39 SW_Push, SW4 SW_Push, SW40 SW_Push, SW41 SW_Push, SW42 SW_Push, SW43 SW_Push, SW44 SW_Push, SW45 SW_Push, SW46 SW_Push, SW47 SW_Push, SW48 SW_Push, SW49 SW_Push, SW5 SW_Push, SW50 SW_Push, SW51 SW_Push, SW52 SW_Push, SW53 SW_Push, SW54 SW_Push, SW55 SW_Push, SW56 SW_Push, SW57 SW_Push, SW58 SW_Push, SW59 SW_Push, SW6 SW_Push, SW60 SW_Push, SW61 SW_Push, SW62 SW_Push, SW7 SW_Push, SW8 SW_Push, SW9 SW_Push, U1 tp4056, U2 PCA9506DGG,512, U3 fs312f, U4 MT3608, U5 PCA9506DGG,512

Commit message: Layout
Parts:
- removed J3: Debug, Connector_PinHeader_2.54mm:PinHeader_1x04_P2.54mm_Vertical
- added U6: nRF52840_dongle, NRF_Dongle:nRF52840_dongle, F.Cu at (198.2, 90.2)
- C1, C2, C3, D1, L1, Q1, R1, R4, R5, R6, R7, U1, U3, U4: moved to B.Cu
- J1: value USB_C_Receptacle -> USB_C_Receptacle_USB2.0; footprint Connector_USB:USB_C_Receptacle_HRO_TYPE-C-31-M-12 -> Connector_USB:USB_C_Receptacle_XKB_U262-16XN-4BVC11
- SW60: footprint Button_Switch_Keyboard:SW_Cherry_MX_2.25u_PCB -> Button_Switch_Keyboard:SW_Cherry_MX_2.00u_PCB
- moved J2 300.0 mm to (341.0, 93.0)
- moved SW59 292.3 mm to (319.2, 163.7)
- moved SW58 288.3 mm to (324.0, 144.6)
- moved U2 268.3 mm to (293.0, 90.0), turned to 180 degrees
- moved SW57 260.7 mm to (309.7, 182.7)
- moved SW62 259.9 mm to (333.5, 182.7)
- moved SW61 254.9 mm to (331.1, 125.5)
- moved SW56 249.0 mm to (307.3, 125.5)
- moved SW49 237.2 mm to (262.1, 182.7)
- moved C1 223.4 mm to (264.1, 89.1), turned to 90 degrees
- moved U1 222.3 mm to (260.7, 88.2), turned to 180 degrees
- moved J4 219.8 mm to (267.7, 82.7)
- moved Q1 218.3 mm to (250.0, 91.6), turned to -90 degrees
- moved R1 217.5 mm to (264.1, 87.2), turned to 90 degrees
- moved C2 215.6 mm to (257.1, 92.4), turned to -90 degrees
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Connections:
- SW4 pad 1: unconnected-(SW4-Pad1) -> /K_CAPLOCK
- U2 pad 10: unconnected-(U2-Pad10) -> /K_I
- U2 pad 12: unconnected-(U2-Pad12) -> /K_K
- U2 pad 13: unconnected-(U2-Pad13) -> /K_BSP
- U2 pad 14: unconnected-(U2-Pad14) -> /K_RETURN
- U2 pad 15: unconnected-(U2-Pad15) -> /K_RALT
- U2 pad 16: unconnected-(U2-Pad16) -> /K_RGUI
- U2 pad 17: unconnected-(U2-Pad17) -> /K_FN
- U2 pad 19: unconnected-(U2-Pad19) -> /K_RSHIFT
- U2 pad 20: unconnected-(U2-Pad20) -> /K_RCTRL
- U2 pad 22: unconnected-(U2-Pad22) -> /K_,
- U2 pad 24: unconnected-(U2-Pad24) -> /K_9
- U2 pad 25: unconnected-(U2-Pad25) -> /K_O
- U2 pad 26: unconnected-(U2-Pad26) -> /K_L
- U2 pad 3: unconnected-(U2-Pad3) -> /K_N
- U2 pad 31: unconnected-(U2-Pad31) -> /K_.
- U2 pad 32: unconnected-(U2-Pad32) -> /K_0
- U2 pad 33: unconnected-(U2-Pad33) -> /K_P
- U2 pad 35: unconnected-(U2-Pad35) -> /K_;
- U2 pad 4: unconnected-(U2-Pad4) -> /K_7
- U2 pad 45: unconnected-(U2-Pad45) -> /K_\/
- U2 pad 47: unconnected-(U2-Pad47) -> /K_-
- U2 pad 48: unconnected-(U2-Pad48) -> /K_\{
- U2 pad 49: unconnected-(U2-Pad49) -> /K_'
- U2 pad 5: unconnected-(U2-Pad5) -> /K_U
- U2 pad 50: unconnected-(U2-Pad50) -> /K_\
- U2 pad 52: unconnected-(U2-Pad52) -> /K_\}
- U2 pad 53: unconnected-(U2-Pad53) -> /K_=
- U2 pad 54: unconnected-(U2-Pad54) -> /K_SPACE
- U2 pad 7: unconnected-(U2-Pad7) -> /K_J
- U2 pad 8: unconnected-(U2-Pad8) -> /K_M
- U2 pad 9: unconnected-(U2-Pad9) -> /K_8
- U5 pad 10: unconnected-(U5-Pad10) -> /K_Q
- U5 pad 12: unconnected-(U5-Pad12) -> /K_A
- U5 pad 13: unconnected-(U5-Pad13) -> /K_T
- U5 pad 14: unconnected-(U5-Pad14) -> /K_G
- U5 pad 15: unconnected-(U5-Pad15) -> /K_B
- U5 pad 16: unconnected-(U5-Pad16) -> /K_6
- U5 pad 17: unconnected-(U5-Pad17) -> /K_Y
- U5 pad 19: unconnected-(U5-Pad19) -> /K_H
- U5 pad 22: unconnected-(U5-Pad22) -> /K_Z
- U5 pad 24: unconnected-(U5-Pad24) -> /K_LGUI
- U5 pad 25: unconnected-(U5-Pad25) -> /K_2
- U5 pad 26: unconnected-(U5-Pad26) -> /K_W
- U5 pad 3: unconnected-(U5-Pad3) -> /K_ESC
- U5 pad 31: unconnected-(U5-Pad31) -> /K_S
- U5 pad 32: unconnected-(U5-Pad32) -> /K_X
- U5 pad 33: unconnected-(U5-Pad33) -> /K_LALT
- U5 pad 35: unconnected-(U5-Pad35) -> /K_3
- U5 pad 4: unconnected-(U5-Pad4) -> /K_TAB
- U5 pad 45: unconnected-(U5-Pad45) -> /K_E
- U5 pad 47: unconnected-(U5-Pad47) -> /K_D
- U5 pad 48: unconnected-(U5-Pad48) -> /K_C
- U5 pad 49: unconnected-(U5-Pad49) -> /K_4
- U5 pad 5: unconnected-(U5-Pad5) -> /K_LCTRL
- U5 pad 50: unconnected-(U5-Pad50) -> /K_R
- U5 pad 52: unconnected-(U5-Pad52) -> /K_F
- U5 pad 53: unconnected-(U5-Pad53) -> /K_V
- U5 pad 54: unconnected-(U5-Pad54) -> /K_5
- U5 pad 7: unconnected-(U5-Pad7) -> /K_LSHIFT
- U5 pad 8: unconnected-(U5-Pad8) -> /K_CAPLOCK
- U5 pad 9: unconnected-(U5-Pad9) -> /K_1
Routing:
- net VBUS: track 0.00 -> 75.3 mm, vias 0 -> 2
- net D-: track 0.00 -> 30.1 mm, vias 0 -> 2
- net D+: track 0.00 -> 29.7 mm
- net -BATT: track 0.00 -> 28.5 mm, vias 0 -> 2
- net +BATT: track 0.00 -> 27.8 mm, vias 0 -> 2
- net +VSW: track 0.00 -> 25.9 mm, vias 0 -> 3
- net Net-(J1-PadB5): track 0.00 -> 12.1 mm, vias 0 -> 2
- net GND: track 0.00 -> 10.2 mm, vias 0 -> 3
- net Net-(J1-PadA5): track 0.00 -> 6.58 mm
- net Net-(D1-Pad2): track 0.00 -> 5.04 mm
- net Net-(C2-Pad1): track 0.00 -> 4.82 mm
- net Net-(Q1-Pad1): track 0.00 -> 4.53 mm
- net Net-(R5-Pad1): track 0.00 -> 4.20 mm
- net Net-(R6-Pad2): track 0.00 -> 3.69 mm
- net Net-(Q1-Pad4): track 0.00 -> 2.41 mm
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- added copper zone on B.Cu, net GND
- added copper zone on F.Cu, net GND
Other:
- board outline added: 288 x 120 mm

Commit message: Routing
Parts:
- removed R10: 4k7, Resistor_SMD:R_0201_0603Metric_Pad0.64x0.40mm_HandSolder
- moved R14 2.58 mm to (194.6, 80.8)
- moved R13 2.56 mm to (192.0, 80.8)
- turned R12 to 0 degrees
- turned U2 to 0 degrees
Connections:
- R11 pad 2: INT1 -> INT2
- R12 pad 2: INT2 -> INT1
- U2 pad 12: /K_K -> /K_M
- U2 pad 13: /K_BSP -> /K_0
- U2 pad 14: /K_RETURN -> /K_K
- U2 pad 15: /K_RALT -> /K_,
- U2 pad 16: /K_RGUI -> /K_O
- U2 pad 17: /K_FN -> /K_L
- U2 pad 19: /K_RSHIFT -> /K_.
- U2 pad 20: /K_RCTRL -> /K_RALT
- U2 pad 21: unconnected-(U2-Pad21) -> /K_RGUI
- U2 pad 22: /K_, -> /K_\/
- U2 pad 24: /K_9 -> /K_;
- U2 pad 25: /K_O -> /K_P
- U2 pad 26: /K_L -> /K_-
- U2 pad 3: /K_N -> /K_7
- U2 pad 31: /K_. -> unconnected-(U2-Pad31)
- U2 pad 32: /K_0 -> unconnected-(U2-Pad32)
- U2 pad 33: /K_P -> unconnected-(U2-Pad33)
- U2 pad 35: /K_; -> unconnected-(U2-Pad35)
- U2 pad 4: /K_7 -> /K_U
- U2 pad 43: unconnected-(U2-Pad43) -> /K_=
- U2 pad 44: unconnected-(U2-Pad44) -> /K_\{
- U2 pad 45: /K_\/ -> /K_'
- U2 pad 47: /K_- -> /K_\}
- U2 pad 48: /K_\{ -> /K_RETURN
- U2 pad 49: /K_' -> /K_\
- U2 pad 5: /K_U -> /K_N
- U2 pad 50: /K_\ -> /K_BSP
- U2 pad 52: /K_\} -> /K_RSHIFT
- U2 pad 53: /K_= -> /K_FN
- U2 pad 54: /K_SPACE -> /K_RCTRL
- U2 pad 55: INT1 -> INT2
- U2 pad 56: RST -> VDD
- U2 pad 8: /K_M -> /K_8
- U2 pad 9: /K_8 -> /K_9
- U5 pad 13: /K_T -> /K_LGUI
- U5 pad 14: /K_G -> /K_Z
- U5 pad 15: /K_B -> /K_LALT
- U5 pad 16: /K_6 -> /K_X
- U5 pad 17: /K_Y -> /K_S
- U5 pad 19: /K_H -> /K_W
- U5 pad 20: unconnected-(U5-Pad20) -> /K_2
- U5 pad 21: unconnected-(U5-Pad21) -> /K_C
- U5 pad 22: /K_Z -> /K_D
- U5 pad 24: /K_LGUI -> /K_E
- U5 pad 25: /K_2 -> /K_3
- U5 pad 26: /K_W -> /K_SPACE
- U5 pad 31: /K_S -> unconnected-(U5-Pad31)
- U5 pad 32: /K_X -> unconnected-(U5-Pad32)
- U5 pad 33: /K_LALT -> unconnected-(U5-Pad33)
- U5 pad 35: /K_3 -> unconnected-(U5-Pad35)
- U5 pad 4: /K_TAB -> /K_LSHIFT
- U5 pad 42: unconnected-(U5-Pad42) -> /K_4
- U5 pad 43: unconnected-(U5-Pad43) -> /K_R
- U5 pad 44: unconnected-(U5-Pad44) -> /K_F
- U5 pad 45: /K_E -> /K_V
- U5 pad 47: /K_D -> /K_5
- U5 pad 48: /K_C -> /K_T
- U5 pad 49: /K_4 -> /K_G
- U5 pad 5: /K_LCTRL -> /K_TAB
- U5 pad 50: /K_R -> /K_B
- U5 pad 52: /K_F -> /K_H
- U5 pad 53: /K_V -> /K_Y
- U5 pad 54: /K_5 -> /K_6
- U5 pad 55: INT2 -> INT1
- U5 pad 56: RST -> VDD
- U5 pad 7: /K_LSHIFT -> /K_LCTRL
- U6 pad 5: INT1 -> INT2
- U6 pad 6: INT2 -> INT1
- U6 pad 7: INT_Ext1 -> INT_Ext2
- U6 pad 8: INT_Ext2 -> INT_Ext1
Routing:
- net SCL: track 0.00 -> 317.0 mm, vias 0 -> 2
- net VDD: track 0.00 -> 294.5 mm, vias 0 -> 9
- net SDA: track 0.00 -> 244.5 mm, vias 0 -> 2
- net INT_Ext2: track 0.00 -> 178.6 mm, vias 0 -> 1
- net INT_Ext1: track 0.00 -> 170.9 mm, vias 0 -> 1
- net /K_FN: track 0.00 -> 155.4 mm
- net /K_SPACE: track 0.00 -> 152.7 mm
- net /K_N: track 0.00 -> 152.2 mm
- net /K_RCTRL: track 0.00 -> 136.9 mm
- net /K_J: track 0.00 -> 126.0 mm
- net /K_B: track 0.00 -> 125.5 mm
- net /K_CAPLOCK: track 0.00 -> 120.8 mm
- net /K_RGUI: track 0.00 -> 120.5 mm
- net /K_RALT: track 0.00 -> 117.1 mm
- net /K_RSHIFT: track 0.00 -> 115.1 mm
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
Commit message: Via Stitching
Routing:
- net GND: vias 21 -> 2996

Commit message: Improve tracing
Parts:
- J2: footprint Connector_PinHeader_1.00mm:PinHeader_1x06_P1.00mm_Vertical -> Connector_PinHeader_1.00mm:PinHeader_1x06_P1.00mm_Horizontal
- moved J2 0.38 mm to (340.6, 93.0)
Routing:
- net SCL: track 317.0 -> 244.2 mm
- net GND: track 36.7 -> 39.1 mm
- net -BATT: track 28.5 -> 30.8 mm
