File: KBLE60.kicad_sch (KiCad schematic)
At the start: 92 parts, among them J1 USB_C_Receptacle, J2 Ext_pin, J3 Debug, J4 Battery, Q1 Q_Dual_NMOS_G1S2G2D2S1D1, SW1 SW_Push, SW10 SW_DPDT_x2, SW11 SW_Push, SW12 SW_Push, SW13 SW_Push, SW14 SW_Push, SW15 SW_Push, SW16 SW_Push, SW17 SW_Push, SW18 SW_Push, SW19 SW_Push, SW2 SW_Push, SW20 SW_Push, SW21 SW_Push, SW22 SW_Push, SW23 SW_Push, SW24 SW_Push, SW25 SW_Push, SW26 SW_Push, SW27 SW_Push, SW28 SW_Push, SW29 SW_Push, SW3 SW_Push, SW30 SW_Push, SW31 SW_Push, SW32 SW_Push, SW33 SW_Push, SW34 SW_Push, SW35 SW_Push, SW36 SW_Push, SW37 SW_Push, SW38 SW_Push, SW39 SW_Push, SW4 SW_Push, SW40 SW_Push, SW41 SW_Push, SW42 SW_Push, SW43 SW_Push, SW44 SW_Push, SW45 SW_Push, SW46 SW_Push, SW47 SW_Push, SW48 SW_Push, SW49 SW_Push, SW5 SW_Push, SW50 SW_Push, SW51 SW_Push, SW52 SW_Push, SW53 SW_Push, SW54 SW_Push, SW55 SW_Push, SW56 SW_Push, SW57 SW_Push, SW58 SW_Push, SW59 SW_Push, SW6 SW_Push, SW60 SW_Push, SW61 SW_Push, SW62 SW_Push, SW7 SW_Push, SW8 SW_Push, SW9 SW_Push, U1 tp4056, U2 PCA9506DGG,512, U3 fs312f, U4 MT3608, U5 PCA9506DGG,512, U6 nRF52840_dongle

Commit message: Layout
Parts:
- removed J1: USB_C_Receptacle, Connector_USB:USB_C_Receptacle_HRO_TYPE-C-31-M-12, symbol Connector:USB_C_Receptacle
- removed J3: Debug, Connector_PinHeader_2.54mm:PinHeader_1x04_P2.54mm_Vertical, symbol Connector:Conn_01x04_Female
- added J1: USB_C_Receptacle_USB2.0, Connector_USB:USB_C_Receptacle_XKB_U262-16XN-4BVC11, symbol Connector:USB_C_Receptacle_USB2.0
- SW60: footprint Button_Switch_Keyboard:SW_Cherry_MX_2.25u_PCB -> Button_Switch_Keyboard:SW_Cherry_MX_2.00u_PCB
- U6: now in the parts list
Connections:
- net D+: now also J1.A6 (D+), J1.B6 (D+)
- net D-: now also J1.A7 (D-), J1.B7 (D-)
- net GND: now also J1.A1 (GND), J1.A12 (GND), J1.B1 (GND), J1.B12 (GND), J1.S1 (SHIELD)
- net K_': now also U2.49 (IO4_3)
- net K_,: now also U2.22 (IO2_0)
- net K_-: now also U2.47 (IO4_1)
- net K_.: now also U2.31 (IO2_4)
- net K_0: now also U2.32 (IO2_5)
- net K_1: now also U5.9 (IO0_5)
- net K_2: now also U5.25 (IO2_2)
- net K_3: now also U5.35 (IO2_7)
- net K_4: now also U5.49 (IO4_3)
- net K_5: now also U5.54 (IO4_7)
- net K_6: now also U5.16 (IO1_3)
- net K_7: now also U2.4 (IO0_1)
- net K_8: now also U2.9 (IO0_5)
- net K_9: now also U2.24 (IO2_1)
- net K_;: now also U2.35 (IO2_7)
- net K_=: now also U2.53 (IO4_6)
- net K_A: now also U5.12 (IO0_7)
- net K_B: now also U5.15 (IO1_2)
- net K_BSP: now also U2.13 (IO1_0)
- net K_C: now also U5.48 (IO4_2)
- net K_CAPLOCK: now also SW4.1, U5.8 (IO0_4)
- net K_D: now also U5.47 (IO4_1)
- net K_E: now also U5.45 (IO4_0)
- net K_ESC: now also U5.3 (IO0_0)
- net K_F: now also U5.52 (IO4_5)
- net K_FN: now also U2.17 (IO1_4)
- net K_G: now also U5.14 (IO1_1)
- net K_H: now also U5.19 (IO1_5)
- net K_I: now also U2.10 (IO0_6)
- net K_J: now also U2.7 (IO0_3)
- net K_K: now also U2.12 (IO0_7)
- net K_L: now also U2.26 (IO2_3)
- net K_LALT: now also U5.33 (IO2_6)
- net K_LCTRL: now also U5.5 (IO0_2)
- net K_LGUI: now also U5.24 (IO2_1)
- net K_LSHIFT: now also U5.7 (IO0_3)
- net K_M: now also U2.8 (IO0_4)
- net K_N: now also U2.3 (IO0_0)
- net K_O: now also U2.25 (IO2_2)
- net K_P: now also U2.33 (IO2_6)
- net K_Q: now also U5.10 (IO0_6)
- net K_R: now also U5.50 (IO4_4)
- net K_RALT: now also U2.15 (IO1_2)
- net K_RCTRL: now also U2.20 (IO1_6)
- net K_RETURN: now also U2.14 (IO1_1)
- net K_RGUI: now also U2.16 (IO1_3)
- net K_RSHIFT: now also U2.19 (IO1_5)
- net K_S: now also U5.31 (IO2_4)
- net K_SPACE: now also U2.54 (IO4_7)
- net K_T: now also U5.13 (IO1_0)
- net K_TAB: now also U5.4 (IO0_1)
- net K_U: now also U2.5 (IO0_2)
- net K_V: now also U5.53 (IO4_6)
- net K_W: now also U5.26 (IO2_3)
- net K_X: now also U5.32 (IO2_5)
- net K_Y: now also U5.17 (IO1_4)
- net K_Z: now also U5.22 (IO2_0)
- net K_\: now also U2.50 (IO4_4)
- net K_\{: now also U2.48 (IO4_2)
- net K_\/: now also U2.45 (IO4_0)
- net K_\}: now also U2.52 (IO4_5)
- net VBUS: now also U6.26 (VBUS), J1.A4 (VBUS), J1.A9 (VBUS), J1.B4 (VBUS), J1.B9 (VBUS)
- net at R3.1: now also J1.A5 (CC1)
- net at R2.1: now also J1.B5 (CC2)
- no-connect marks 24 -> 35
Other:
- moved on the sheet: U2A, U2B, U5A, U5B

Commit message: Routing
Parts:
- removed R10: 4k7, Resistor_SMD:R_0201_0603Metric_Pad0.64x0.40mm_HandSolder, symbol Device:R_Small
Connections:
- net RST is gone; now on net VDD: U2.56 (~{RESET}), U5.56 (~{RESET})
- net INT1: now also R12.2, U5.55 (~{INT}), U6.6 (P0.22); no longer R11.2, U2.55 (~{INT}), U6.5 (P0.20)
- net INT2: now also R11.2, U2.55 (~{INT}), U6.5 (P0.20); no longer R12.2, U5.55 (~{INT}), U6.6 (P0.22)
- net INT_Ext1: now also U6.8 (P1.00); no longer U6.7 (P0.24)
- net INT_Ext2: now also U6.7 (P0.24); no longer U6.8 (P1.00)
- net K_': now also U2.45 (IO4_0); no longer U2.49 (IO4_3)
- net K_,: now also U2.15 (IO1_2); no longer U2.22 (IO2_0)
- net K_-: now also U2.26 (IO2_3); no longer U2.47 (IO4_1)
- net K_.: now also U2.19 (IO1_5); no longer U2.31 (IO2_4)
- net K_0: now also U2.13 (IO1_0); no longer U2.32 (IO2_5)
- net K_2: now also U5.20 (IO1_6); no longer U5.25 (IO2_2)
- net K_3: now also U5.25 (IO2_2); no longer U5.35 (IO2_7)
- net K_4: now also U5.42 (IO3_5); no longer U5.49 (IO4_3)
- net K_5: now also U5.47 (IO4_1); no longer U5.54 (IO4_7)
- net K_6: now also U5.54 (IO4_7); no longer U5.16 (IO1_3)
- net K_7: now also U2.3 (IO0_0); no longer U2.4 (IO0_1)
- net K_8: now also U2.8 (IO0_4); no longer U2.9 (IO0_5)
- net K_9: now also U2.9 (IO0_5); no longer U2.24 (IO2_1)
- net K_;: now also U2.24 (IO2_1); no longer U2.35 (IO2_7)
- net K_=: now also U2.43 (IO3_6); no longer U2.53 (IO4_6)
- net K_B: now also U5.50 (IO4_4); no longer U5.15 (IO1_2)
- net K_BSP: now also U2.50 (IO4_4); no longer U2.13 (IO1_0)
- net K_C: now also U5.21 (IO1_7); no longer U5.48 (IO4_2)
- net K_D: now also U5.22 (IO2_0); no longer U5.47 (IO4_1)
- net K_E: now also U5.24 (IO2_1); no longer U5.45 (IO4_0)
- net K_F: now also U5.44 (IO3_7); no longer U5.52 (IO4_5)
- net K_FN: now also U2.53 (IO4_6); no longer U2.17 (IO1_4)
- net K_G: now also U5.49 (IO4_3); no longer U5.14 (IO1_1)
- net K_H: now also U5.52 (IO4_5); no longer U5.19 (IO1_5)
- net K_K: now also U2.14 (IO1_1); no longer U2.12 (IO0_7)
- net K_L: now also U2.17 (IO1_4); no longer U2.26 (IO2_3)
- net K_LALT: now also U5.15 (IO1_2); no longer U5.33 (IO2_6)
- net K_LCTRL: now also U5.7 (IO0_3); no longer U5.5 (IO0_2)
- net K_LGUI: now also U5.13 (IO1_0); no longer U5.24 (IO2_1)
- net K_LSHIFT: now also U5.4 (IO0_1); no longer U5.7 (IO0_3)
- net K_M: now also U2.12 (IO0_7); no longer U2.8 (IO0_4)
- net K_N: now also U2.5 (IO0_2); no longer U2.3 (IO0_0)
- net K_O: now also U2.16 (IO1_3); no longer U2.25 (IO2_2)
- net K_P: now also U2.25 (IO2_2); no longer U2.33 (IO2_6)
- net K_R: now also U5.43 (IO3_6); no longer U5.50 (IO4_4)
- net K_RALT: now also U2.20 (IO1_6); no longer U2.15 (IO1_2)
- net K_RCTRL: now also U2.54 (IO4_7); no longer U2.20 (IO1_6)
- net K_RETURN: now also U2.48 (IO4_2); no longer U2.14 (IO1_1)
- net K_RGUI: now also U2.21 (IO1_7); no longer U2.16 (IO1_3)
- net K_RSHIFT: now also U2.52 (IO4_5); no longer U2.19 (IO1_5)
- net K_S: now also U5.17 (IO1_4); no longer U5.31 (IO2_4)
- net K_SPACE: now also U5.26 (IO2_3); no longer U2.54 (IO4_7)
- net K_T: now also U5.48 (IO4_2); no longer U5.13 (IO1_0)
- net K_TAB: now also U5.5 (IO0_2); no longer U5.4 (IO0_1)
- net K_U: now also U2.4 (IO0_1); no longer U2.5 (IO0_2)
- net K_V: now also U5.45 (IO4_0); no longer U5.53 (IO4_6)
- net K_W: now also U5.19 (IO1_5); no longer U5.26 (IO2_3)
- net K_X: now also U5.16 (IO1_3); no longer U5.32 (IO2_5)
- net K_Y: now also U5.53 (IO4_6); no longer U5.17 (IO1_4)
- net K_Z: now also U5.14 (IO1_1); no longer U5.22 (IO2_0)
- net K_\: now also U2.49 (IO4_3); no longer U2.50 (IO4_4)
- net K_\{: now also U2.44 (IO3_7); no longer U2.48 (IO4_2)
- net K_\/: now also U2.22 (IO2_0); no longer U2.45 (IO4_0)
- net K_\}: now also U2.47 (IO4_1); no longer U2.52 (IO4_5)
- no-connect marks 35 -> 25

Commit message: Improve tracing
Parts:
- J2: footprint Connector_PinHeader_1.00mm:PinHeader_1x06_P1.00mm_Vertical -> Connector_PinHeader_1.00mm:PinHeader_1x06_P1.00mm_Horizontal
Changed lines of the file:
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@@
       (effects (font (size 1.27 1.27)) (justify left))
     )
-    (property "Footprint" "Connector_PinHeader_1.00mm:PinHeader_1x06_P1.00mm_Vertical" (id 2) (at 325.12 34.29 0)
+    (property "Footprint" "Connector_PinHeader_1.00mm:PinHeader_1x06_P1.00mm_Horizontal" (id 2) (at 325.12 34.29 0)
       (effects (font (size 1.27 1.27)) hide)
     )
@@
     )
     (path "/58e4e739-52d2-48d7-88dd-c2bdbef2a23e"
-      (reference "J2") (unit 1) (value "Ext_pin") (footprint "Connector_PinHeader_1.00mm:PinHeader_1x06_P1.00mm_Vertical")
+      (reference "J2") (unit 1) (value "Ext_pin") (footprint "Connector_PinHeader_1.00mm:PinHeader_1x06_P1.00mm_Horizontal")
     )
     (path "/6ad476f6-8d94-4749-8190-59571119ea6b"
